File: kicad/v1.0/keyboard/Key.kicad_sch (KiCad schematic)
At the start: 2 parts, among them SW2 KeyButton

Commit message: Positioning
- Added Library
- Created Footprint for 2-pin push-button
- Added additional keys for ENTER and SPACE to cover whole length
- Added keys for numpad (1:1 link to other number keys)
- Positioned main keys, numpad keys
- Created cutout for reset switch
Parts:
- SW2: footprint Button_Switch_THT:SW_PUSH_6mm -> Library:SW_SPST_Push
