File: kicad/v1.0/pp/TRS-IO++.kicad_sch (KiCad schematic)
At the start: 90 parts, among them J1 Conn_02x06_Odd_Even, J13 UART, J2 Interface Connector, J3 TRS-80 M3 Edge Connector, J4 SPEAKER, J5 Conn_02x06_Odd_Even, J6 LED3, J7 HDMI, J8 Programmer, J9 LED4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

Commit message: Add trimpot part number
Parts:
- RV1: LCSC (none) -> C720648
Changed lines of the file:
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@@
+			)
+		)
+		(property "LCSC" "C720648"
+			(at 381 58.42 0)
+			(effects
+				(font
+					(size 1.27 1.27)
+				)
+				(hide yes)
 			)
 		)
