File: kicad/v1.1/pp/TRS-IO++.kicad_pcb (KiCad board)
At the start: 2 copper layers, 145.7 x 88.6 mm, 89 parts, among them J1 Conn_02x06_Odd_Even, J10 Conn_01x08, J13 UART, J2 Interface Connector, J3 TRS-80 M3 Edge Connector, J4 SPEAKER, J5 Conn_02x06_Odd_Even, J6 LED3, J7 HDMI, J8 Programmer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

Commit message: V1.1 of PCB
Parts:
- RV1: footprint Potentiometer_SMD:Potentiometer_Bourns_TC33X_Vertical -> Potentiometer_THT:Potentiometer_Bourns_3266W_Vertical
- moved RV1 30.9 mm to (202.4, 70.3), turned to 90 degrees
- moved C16 14.8 mm to (180.6, 66.2)
- moved R18 14.8 mm to (178.3, 66.2)
- moved J4 12.3 mm to (194.2, 71.5), turned to 180 degrees
- moved C22 2.63 mm to (176.0, 71.1)
- moved R16 2.63 mm to (178.3, 71.0)
- moved C27 2.07 mm to (176.0, 66.3)
- moved R31 2.07 mm to (173.8, 66.3)
Routing:
- net Net-(C16-Pad2): track 2.97 -> 31.4 mm
- net Net-(C22-Pad1): track 4.77 -> 30.8 mm
- net Net-(J4-Pin_1): track 15.5 -> 32.6 mm
- net Net-(U4--): track 16.7 -> 8.83 mm
- net Net-(J4-Pin_2): track 29.6 -> 35.9 mm
- net GND: track 262.2 -> 259.8 mm, vias 50 -> 51
- net CASS_OUT: track 148.3 -> 149.6 mm
Other:
- board text added: "MiniTRS-M3 V1.1 February 2026"
- board text removed: "MiniTRS-M3 V1.1 October 2025"
