File: kicad/v1.1/pp/TRS-IO++.kicad_sch (KiCad schematic)
At the start: 89 parts, among them J1 Conn_02x06_Odd_Even, J10 Conn_01x08, J13 UART, J2 Interface Connector, J3 TRS-80 M3 Edge Connector, J4 SPEAKER, J5 Conn_02x06_Odd_Even, J6 LED3, J7 HDMI, J8 Programmer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

Commit message: V1.1 of PCB
Parts:
- RV1: footprint Potentiometer_SMD:Potentiometer_Bourns_TC33X_Vertical -> Potentiometer_THT:Potentiometer_Bourns_3266W_Vertical; LCSC C720648 -> C123864
Changed lines of the file:
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@@
 			)
 		)
-		(property "Footprint" "Potentiometer_SMD:Potentiometer_Bourns_TC33X_Vertical"
+		(property "Footprint" "Potentiometer_THT:Potentiometer_Bourns_3266W_Vertical"
 			(at 381 58.42 0)
 			(effects
@@
 			)
 		)
-		(property "LCSC" "C720648"
+		(property "LCSC" "C123864"
 			(at 381 58.42 0)
 			(effects
